Commit message: Load SImulation Testing Added

File: lower_body.urdf (robot description, URDF)
Before this commit: robot onshape, 11 links, 10 joints
Links:
- link foot: geometry collision mesh filename=objects/foot_collision.obj; visual mesh filename=objects/foot_visual.obj
- link foot_2: geometry collision mesh filename=objects/foot_2_collision.obj; visual mesh filename=objects/foot_2_visual.obj
- link hip_pitch: geometry collision mesh filename=objects/hip_pitch_collision.obj; visual mesh filename=objects/hip_pitch_visual.obj
- link hip_pitch_2: geometry collision mesh filename=objects/hip_pitch_2_collision.obj; visual mesh filename=objects/hip_pitch_2_visual.obj
- link hip_roll: geometry collision mesh filename=objects/hip_roll_collision.obj; visual mesh filename=objects/hip_roll_visual.obj
- link hip_roll_2: geometry collision mesh filename=objects/hip_roll_2_collision.obj; visual mesh filename=objects/hip_roll_2_visual.obj
- link lower_leg: geometry collision mesh filename=objects/lower_leg_collision.obj; visual mesh filename=objects/lower_leg_visual.obj
- link lower_leg_2: geometry collision mesh filename=objects/lower_leg_2_collision.obj; visual mesh filename=objects/lower_leg_2_visual.obj
- link pelvis: geometry collision mesh filename=objects/pelvis_collision.obj; visual mesh filename=objects/pelvis_visual.obj
- link upper_leg: geometry collision mesh filename=objects/upper_leg_collision.obj; visual mesh filename=objects/upper_leg_visual.obj
- link upper_leg_2: geometry collision mesh filename=objects/upper_leg_2_collision.obj; visual mesh filename=objects/upper_leg_2_visual.obj
