Commit message: Testing global IK on fast computer.

File: lower_body_modified.urdf (robot description, URDF)
Before this commit: robot onshape, 11 links, 10 joints
Joints:
- joint L_hip_pitch: origin xyz=-0.059000000000000010769 0.062399999999999997136 -0.022499999999999992228 rpy=-1.570796326794896558 7.6605388699134444448e-15 3.1415926535897789051 -> xyz=-0.059000000000000010769 0.062399999999999997136 -0.022499999999999992228 rpy=0 0 0
- joint L_hip_roll: origin xyz=0.062000000000000186906 1.3877787807814456755e-17 -0.069000000000000061284 rpy=2.0954117794914131481e-30 1.5707963267948823471 0 -> xyz=0.062000000000000186906 1.3877787807814456755e-17 -0.069000000000000061284 rpy=0 0 0
- joint L_hip_yaw: origin xyz=2.7755575615628913511e-17 0.030699999999999963429 -0.061999999999999985678 rpy=1.570796326794896558 -3.1469101559397065552e-14 5.5511151231126851459e-17 -> xyz=2.7755575615628913511e-17 0.030699999999999963429 -0.061999999999999985678 rpy=0 0 0
- joint R_hip_pitch: origin xyz=-0.05900000000000000383 -0.062400000000000011013 -0.022499999999999992228 rpy=1.570796326794896558 -1.8873791418627657243e-15 -3.1415926535897895633 -> xyz=-0.05900000000000000383 -0.062400000000000011013 -0.022499999999999992228 rpy=1.57 0 0
- joint R_hip_roll: origin xyz=0.061999999999999992617 3.4694469519536141888e-18 -0.069000000000000019651 rpy=-3.141592653589793116 -1.5707963267948930053 0 -> xyz=0.061999999999999992617 3.4694469519536141888e-18 -0.069000000000000019651 rpy=0 1.57 0
- joint R_hip_yaw: origin xyz=0 0.03069999999999989404 -0.061999999999999978739 rpy=1.570796326794896558 -3.1530333899353865146e-14 5.5511151231574739564e-17 -> xyz=0 0.03069999999999989404 -0.061999999999999978739 rpy=0 0 0
